File: MECB_Template_16V8/MECB_Template_16V8.kicad_sch (KiCad schematic)
At the start: 7 parts, among them J1 MECB_64AC, U1 ATF16V8

Commit message: MECB_Template_16V8 / MECB_Template_22V10 - Update (correct) label & net references for active low signals.
Connections:
- net CS0 renamed 0_~{CS}
- net CS1 renamed 1_~{CS}
- net CS2 renamed 2_~{CS}
- net ECB_INT renamed ECB_~{INT}
- net ECB_IORQ renamed ECB_~{IORQ}
- net ECB_MREQ renamed ECB_~{MREQ}
- net ECB_NMI renamed ECB_~{NMI}
- net ECB_RD renamed ECB_~{RD}
- net ECB_RESET renamed ECB_~{RESET}
- net ECB_WR renamed ECB_~{WR}
